Commit message: Created gazebo world that replicated Yongin Driver's License Test Center

File: install/auto_vehicle/share/auto_vehicle/urdf/vehicle.xacro (robot description, xacro)
@@ -1,638 +1 @@
-<?xml version="1.0"?>
-<robot name="ackermann_steering_vehicle" xmlns:xacro="http://www.ros.org/wiki/xacro">
-  <!-- Arguments -->
-  <xacro:arg name="body_length" default="2.0" />
-  <xacro:arg name="body_width" default="1.0" />
-  <xacro:arg name="body_height" default="0.5" />
-  <xacro:arg name="body_density" default="1000.0" />
-  <xacro:arg name="wheel_radius" default="0.3" />
-  <xacro:arg name="wheel_width" default="0.1" />
-  <xacro:arg name="wheel_density" default="1000.0" />
-  <xacro:arg name="max_steering_angle" default="0.6108" />
-  <xacro:arg name="max_steering_angular_velocity" default="1.570796" />
-  <xacro:arg name="max_steering_effort" default="1.0" />
-  <xacro:arg name="max_velocity" default="1.0" />
-  <xacro:arg name="max_effort" default="10.0" />
-  <xacro:arg name="camera_box_size" default="0.1" />
-  <xacro:arg name="camera_stick_size" default="0.2" />
-  <xacro:arg name="camera_height" default="1.5" />
-  <xacro:arg name="camera_pitch" default="0.1" />
-  <xacro:arg name="camera_fov" default="1.396263" />
-  <xacro:arg name="camera_fps" default="30" />
-  <xacro:arg name="image_width" default="640" />
-  <xacro:arg name="image_height" default="480" />
-  <!-- Mathematical Constants -->
-  <xacro:property name="PI" value="3.14159265"/>
-  <!-- Vehicle Properties -->
-  <xacro:property name="body_length" value="$(arg body_length)"/>
-  <xacro:property name="body_width" value="$(arg body_width)"/>
-  <xacro:property name="body_height" value="$(arg body_height)"/>
-  <xacro:property name="body_density" value="$(arg body_density)"/>
-  <xacro:property name="wheel_radius" value="$(arg wheel_radius)"/>
-  <xacro:property name="wheel_width" value="$(arg wheel_width)"/>
-  <xacro:property name="wheel_density" value="$(arg wheel_density)"/>
-  <xacro:property name="max_steering_angle" value="$(arg max_steering_angle)"/>
-  <xacro:property name="max_steering_angular_velocity" value="$(arg max_steering_angular_velocity)"/>
-  <xacro:property name="max_steering_effort" value="$(arg max_steering_effort)"/>
-  <xacro:property name="max_velocity" value="$(arg max_velocity)"/>
-  <xacro:property name="max_effort" value="$(arg max_effort)"/>
-  <xacro:property name="camera_box_size" value="$(arg camera_box_size)"/>
-  <xacro:property name="camera_stick_size" value="$(arg camera_stick_size)"/>
-  <xacro:property name="camera_height" value="$(arg camera_height)"/>
-  <xacro:property name="camera_pitch" value="$(arg camera_pitch)"/>
-  <xacro:property name="camera_fov" value="$(arg camera_fov)"/>
-  <xacro:property name="camera_fps" value="$(arg camera_fps)"/>
-  <xacro:property name="image_width" value="$(arg image_width)"/>
-  <xacro:property name="image_height" value="$(arg image_height)"/>
-  <xacro:property name="body_mass" value="${body_density * body_length * body_height * body_width}"/>
-  <xacro:property name="body_inertia_x" value="${1.0/12.0 * body_mass * (body_height*body_height + body_width*body_width)}"/>
-  <xacro:property name="body_inertia_y" value="${1.0/12.0 * body_mass * (body_length*body_length + body_height*body_height)}"/>
-  <xacro:property name="body_inertia_z" value="${1.0/12.0 * body_mass * (body_length*body_length + body_width*body_width)}"/>
-  <xacro:property name="wheel_separation" value="${body_width + wheel_width}"/>
-  <xacro:property name="wheel_offset" value="${body_length/2 - wheel_radius}"/>
-  <xacro:property name="wheel_mass" value="${wheel_density * PI * wheel_radius * wheel_radius * wheel_width}"/>
-  <xacro:property name="wheel_inertia_x" value="${1.0/12.0 * wheel_mass * (3*wheel_radius*wheel_radius + wheel_width*wheel_width)}"/>
-  <xacro:property name="wheel_inertia_y" value="${1.0/12.0 * wheel_mass * (3*wheel_radius*wheel_radius + wheel_width*wheel_width)}"/>
-  <xacro:property name="wheel_inertia_z" value="${1.0/2.0 * wheel_mass * wheel_radius * wheel_radius}"/>
-  <xacro:property name="max_wheel_angular_velocity" value="${max_velocity / wheel_radius}"/>
-  <!-- Links -->
-  <!-- Body Link -->
-  <link name="body_link">
-    <visual>
-      <origin xyz="0.0 0.0 0.0" rpy="0.0 0.0 0.0"/>
-      <geometry>
-        <box size="${body_length} ${body_width} ${body_height}"/>
-      </geometry>
-      <material name="body_material">
-        <color rgba="0.25 0.25 0.25 1.0"/>
-      </material>
-    </visual>
-    <collision>
-      <origin xyz="0.0 0.0 0.0" rpy="0.0 0.0 0.0"/>
-      <geometry>
-        <box size="${body_length} ${body_width} ${body_height}"/>
-      </geometry>
-    </collision>
-    <inertial>
-      <mass value="${body_mass}"/>
-      <inertia ixx="${body_inertia_x}" ixy="0.0" ixz="0.0" iyy="${body_inertia_y}" iyz="0" izz="${body_inertia_z}"/>
-      <origin xyz="0 0 0" rpy="0 0 0"/>
-    </inertial>
-  </link>
-  <!-- Front Left Wheel -->
-  <link name="front_left_wheel_link">
-    <visual>
-      <origin xyz="0.0 0.0 0.0" rpy="1.570795 0.0 0.0"/>
-      <geometry>
-        <cylinder radius="${wheel_radius}" length="${wheel_width}"/>
-      </geometry>
-      <material name="wheel_material">
-        <color rgba="0.0 0.0 0.0 1.0"/>
-      </material>
-    </visual>
-    <collision>
-      <origin xyz="0.0 0.0 0.0" rpy="1.570795 0.0 0.0"/>
-      <geometry>
-        <cylinder radius="${wheel_radius}" length="${wheel_width}"/>
-      </geometry>
-    </collision>
-    <inertial>
-      <mass value="${wheel_mass}"/>
-      <inertia ixx="${wheel_inertia_x}" ixy="0.0" ixz="0.0" iyy="${wheel_inertia_y}" iyz="0" izz="${wheel_inertia_z}"/>
-      <origin xyz="0.0 0.0 0.0" rpy="1.570795 0.0 0.0"/>
-    </inertial>
-  </link>
-    <!-- Front Left Wheel Steering -->
-  <link name="front_left_steering_link">
-    <visual>
-      <origin xyz="0.0 0.0 0.0" rpy="1.570795 0.0 0.0"/>
-      <geometry>
-        <cylinder length="0.001" radius="0.01"/>
-      </geometry>
-      <material name="wheel_material">
-        <color rgba="0.0 0.0 0.0 1.0"/>
-      </material>
-    </visual>
-    <collision>
-      <origin xyz="0.0 0.0 0.0" rpy="1.570795 0.0 0.0"/>
-      <geometry>
-        <cylinder length="0.001" radius="0.01"/>
-      </geometry>
-    </collision>
-    <inertial>
-      <mass value="0.01"/>
-      <inertia ixx="0.0" ixy="0.0" ixz="0.0" iyy="0.0" iyz="0.0" izz="0.0"/>
-      <origin xyz="0.0 0.0 0.0" rpy="1.570795 0.0 0.0"/>
-    </inertial>
-  </link>
-  <!-- Front Right Wheel -->
-  <link name="front_right_wheel_link">
-    <visual>
-      <origin xyz="0.0 0.0 0.0" rpy="1.570795 0.0 0.0"/>
-      <geometry>
-        <cylinder radius="${wheel_radius}" length="${wheel_width}"/>
-      </geometry>
-      <material name="wheel_material">
-        <color rgba="0.0 0.0 0.0 1.0"/>
-      </material>
-    </visual>
-    <collision>
-      <origin xyz="0.0 0.0 0.0" rpy="1.570795 0.0 0.0"/>
-      <geometry>
-        <cylinder radius="${wheel_radius}" length="${wheel_width}"/>
-      </geometry>
-    </collision>
-    <inertial>
-      <mass value="${wheel_mass}"/>
-      <inertia ixx="${wheel_inertia_x}" ixy="0.0" ixz="0.0" iyy="${wheel_inertia_y}" iyz="0" izz="${wheel_inertia_z}"/>
-      <origin xyz="0.0 0.0 0.0" rpy="1.570795 0.0 0.0"/>
-    </inertial>
-  </link>
-  <!-- Front Right Wheel Steering -->
-  <link name="front_right_steering_link">
-    <visual>
-      <origin xyz="0.0 0.0 0.0" rpy="1.570795 0.0 0.0"/>
-      <geometry>
-        <cylinder length="0.001" radius="0.01"/>
-      </geometry>
-      <material name="wheel_material">
-        <color rgba="0.0 0.0 0.0 1.0"/>
-      </material>
-    </visual>
-    <collision>
-      <origin xyz="0.0 0.0 0.0" rpy="1.570795 0.0 0.0"/>
-      <geometry>
-        <cylinder length="0.001" radius="0.01"/>
-      </geometry>
-    </collision>
-    <inertial>
-      <mass value="0.01"/>
-      <inertia ixx="0.0" ixy="0.0" ixz="0.0" iyy="0.0" iyz="0.0" izz="0.0"/>
-      <origin xyz="0.0 0.0 0.0" rpy="1.570795 0.0 0.0"/>
-    </inertial>
-  </link>
-  <!-- Rear Left Wheel -->
-  <link name="rear_left_wheel_link">
-    <visual>
-      <origin xyz="0.0 0.0 0.0" rpy="1.570795 0.0 0.0"/>
-      <geometry>
-        <cylinder radius="${wheel_radius}" length="${wheel_width}"/>
-      </geometry>
-      <material name="wheel_material">
-        <color rgba="0.0 0.0 0.0 1.0"/>
-      </material>
-    </visual>
-    <collision>
-      <origin xyz="0.0 0.0 0.0" rpy="1.570795 0.0 0.0"/>
-      <geometry>
-        <cylinder radius="${wheel_radius}" length="${wheel_width}"/>
-      </geometry>
-    </collision>
-    <inertial>
-      <mass value="2"/>
-      <inertia ixx="${wheel_inertia_x}" ixy="0.0" ixz="0.0" iyy="${wheel_inertia_y}" iyz="0" izz="${wheel_inertia_z}"/>
-      <origin xyz="0.0 0.0 0.0" rpy="1.570795 0.0 0.0"/>
-    </inertial>
-  </link>
-  <!-- Rear Right Wheel -->
-  <link name="rear_right_wheel_link">
-    <visual>
-      <origin xyz="0.0 0.0 0.0" rpy="1.570795 0.0 0.0"/>
-      <geometry>
-        <cylinder radius="${wheel_radius}" length="${wheel_width}"/>
-      </geometry>
-      <material name="wheel_material">
-        <color rgba="0.0 0.0 0.0 1.0"/>
-      </material>
-    </visual>
-    <collision>
-      <origin xyz="0.0 0.0 0.0" rpy="1.570795 0.0 0.0"/>
-      <geometry>
-        <cylinder radius="${wheel_radius}" length="${wheel_width}"/>
-      </geometry>
-    </collision>
-    <inertial>
-      <mass value="2"/>
-      <inertia ixx="${wheel_inertia_x}" ixy="0.0" ixz="0.0" iyy="${wheel_inertia_y}" iyz="0" izz="${wheel_inertia_z}"/>
-      <origin xyz="0.0 0.0 0.0" rpy="1.570795 0.0 0.0"/>
-    </inertial>
-  </link>
-  <!-- Camera Stick Link -->
-  <link name="camera_stick_link">
-    <collision>
-      <origin xyz="0 0 0" rpy="0 0 0"/>
-      <geometry>
-        <box size="${camera_stick_size} ${camera_stick_size} ${camera_height}"/>
-      </geometry>
-    </collision>
-    <visual>
-      <origin xyz="0 0 0" rpy="0 0 0"/>
-      <geometry>
-        <box size="${camera_stick_size} ${camera_stick_size} ${camera_height}"/>
-      </geometry>
-      <material name="camera_stick_material">
-        <color rgba="0.25 0.25 0.25 1.0"/>
-      </material>
-    </visual>
-    <inertial>
-      <mass value="1e-5" />
-      <origin xyz="0 0 0" rpy="0 0 0"/>
-      <inertia ixx="1e-6" ixy="0" ixz="0" iyy="1e-6" iyz="0" izz="1e-6" />
-    </inertial>
-  </link>
-  <!-- Camera Link -->
-  <link name="camera_link">
-    <collision>
-      <origin xyz="0 0 0" rpy="0 0 0"/>
-      <geometry>
-        <box size="${camera_box_size} ${camera_box_size} ${camera_box_size}"/>
-      </geometry>
-    </collision>
-    <visual>
-      <origin xyz="0 0 0" rpy="0 0 0"/>
-      <geometry>
-        <box size="${camera_box_size} ${camera_box_size} ${camera_box_size}"/>
-      </geometry>
-      <material name="camera_material">
-        <color rgba="0.0 0.0 0.0 1.0"/>
-      </material>
-    </visual>
-    <inertial>
-      <mass value="1e-5" />
-      <origin xyz="0 0 0" rpy="0 0 0"/>
-      <inertia ixx="1e-6" ixy="0" ixz="0" iyy="1e-6" iyz="0" izz="1e-6" />
-    </inertial>
-  </link>
-  <link name="lidar_link">
-    <visual>
-      <origin xyz="0 0 0" rpy="0 0 0"/>
-      <geometry>
-        <cylinder radius="0.06" length="0.05"/>
-      </geometry>
-      <material name="lidar_material">
-        <color rgba="0.1 0.1 0.1 1.0"/>
-      </material>
-    </visual>
-    <collision>
-      <origin xyz="0 0 0" rpy="0 0 0"/>
-      <geometry>
-        <cylinder radius="0.06" length="0.05"/>
-      </geometry>
-    </collision>
-    <inertial>
-      <mass value="0.1"/>
-      <origin xyz="0 0 0" rpy="0 0 0"/>
-      <inertia ixx="1e-4" ixy="0" ixz="0" iyy="1e-4" iyz="0" izz="1e-4"/>
-    </inertial>
-  </link>
-  <link name="gps_link">
-    <visual>
-      <origin xyz="0 0 0" rpy="0 0 0"/>
-      <geometry>
-        <box size="0.08 0.08 0.03"/>
-      </geometry>
-      <material name="gps_material">
-        <color rgba="0.0 0.3 1.0 1.0"/>
-      </material>
-    </visual>
-    <collision>
-      <origin xyz="0 0 0" rpy="0 0 0"/>
-      <geometry>
-        <box size="0.08 0.08 0.03"/>
-      </geometry>
-    </collision>
-    <inertial>
-      <mass value="0.05"/>
-      <origin xyz="0 0 0" rpy="0 0 0"/>
-      <inertia ixx="1e-5" ixy="0" ixz="0" iyy="1e-5" iyz="0" izz="1e-5"/>
-    </inertial>
-  </link>
-<!-- GPS Fixed Joint -->
-  <joint name="gps_joint" type="fixed">
-    <origin xyz="0 0 ${body_height/2 + 0.25}" rpy="0 0 0"/>
-    <parent link="body_link"/>
-    <child link="gps_link"/>
-  </joint>
-<!-- LiDAR Fixed Joint -->
-  <joint name="lidar_joint" type="fixed">
-    <origin xyz="0.15 0 ${body_height/2 + 0.25}" rpy="0 0 0"/>
-    <parent link="body_link"/>
-    <child link="lidar_link"/>
-  </joint>
-  <!-- Joints -->
-  <!-- Front Left Steering Joint -->
-  <joint name="front_left_steering_joint" type="revolute">
-    <origin xyz="${wheel_offset} ${wheel_separation/2} -${wheel_radius/2}" rpy="0 0 0"/>
-    <parent link="body_link"/>
-    <child link="front_left_steering_link"/>
-    <axis xyz="0 0 1"/>
-    <limit effort="${max_steering_effort}" lower="${-max_steering_angle}" upper="${max_steering_angle}" velocity="${max_steering_angular_velocity}"/>
-    <dynamics damping="0.1" friction="0.1"/>
-  </joint>
-  <!-- Front Left Wheel Joint -->
-  <joint name="front_left_wheel_joint" type="continuous">
-    <origin xyz="0 0 0" rpy="0 0 0"/>
-    <parent link="front_left_steering_link"/>
-    <child link="front_left_wheel_link"/>
-    <axis xyz="0 1 0"/>
-    <limit effort="${max_effort}" velocity="${max_wheel_angular_velocity}"/>
-    <dynamics damping="0.1" friction="0.1"/>
-  </joint>
-  <!-- Front Right Steering Joint -->
-  <joint name="front_right_steering_joint" type="revolute">
-    <origin xyz="${wheel_offset} ${-wheel_separation/2} -${wheel_radius/2}" rpy="0 0 0"/>
-    <parent link="body_link"/>
-    <child link="front_right_steering_link"/>
-    <axis xyz="0 0 1"/>
-    <limit effort="${max_steering_effort}" lower="${-max_steering_angle}" upper="${max_steering_angle}" velocity="${max_steering_angular_velocity}"/>
-    <dynamics damping="0.1" friction="0.1"/>
-  </joint>
-  <!-- Front Right Wheel Joint -->
-  <joint name="front_right_wheel_joint" type="continuous">
-    <origin xyz="0 0 0" rpy="0 0 0"/>
-    <parent link="front_right_steering_link"/>
-    <child link="front_right_wheel_link"/>
-    <axis xyz="0 1 0"/>
-    <limit effort="${max_effort}" velocity="${max_wheel_angular_velocity}"/>
-    <dynamics damping="0.1" friction="0.1"/>
-  </joint>
-  <!-- Rear Left Wheel Joint -->
-  <joint name="rear_left_wheel_joint" type="continuous">
-    <origin xyz="-${wheel_offset} ${wheel_separation/2} -${wheel_radius/2}" rpy="0 0 0"/>
-    <parent link="body_link"/>
-    <child link="rear_left_wheel_link"/>
-    <axis xyz="0 1 0"/>
-    <limit effort="${max_effort}" velocity="${max_wheel_angular_velocity}"/>
-    <dynamics damping="0.1" friction="0.1"/>
-  </joint>
-  <!-- Rear Right Wheel Joint -->
-  <joint name="rear_right_wheel_joint" type="continuous">
-    <origin xyz="-${wheel_offset} ${-wheel_separation/2} -${wheel_radius/2}" rpy="0 0 0"/>
-    <parent link="body_link"/>
-    <child link="rear_right_wheel_link"/>
-    <axis xyz="0 1 0"/>
-    <limit effort="${max_effort}" velocity="${max_wheel_angular_velocity}"/>
-    <dynamics damping="0.1" friction="0.1"/>
-  </joint>
-  <!-- Camera Stick Joint -->
-  <joint name="camera_stick_joint" type="fixed">
-    <axis xyz="0 1 0" />
-    <origin xyz="${body_length/2 - camera_stick_size/2} ${camera_box_size/2 + camera_stick_size/2} ${camera_height/2}" rpy="0.0 0.0 0.0"/>
-    <parent link="body_link"/>
-    <child link="camera_stick_link"/>
-  </joint>
-  <!-- Camera Joint -->
-  <joint name="camera_joint" type="fixed">
-    <axis xyz="0 1 0" />
-    <origin xyz="0.0 ${-camera_box_size/2 - camera_stick_size/2} ${camera_height/2}" rpy="0 ${camera_pitch} 0"/>
-    <parent link="camera_stick_link"/>
-    <child link="camera_link"/>
-  </joint>
-  <gazebo reference="body_link">
-    <mu1>0.0001</mu1>
-    <mu2>0.0001</mu2>
-  </gazebo>
-  <gazebo reference="front_right_wheel_link">
-    <mu1>100.0</mu1>
-    <mu2>100.0</mu2>
-  </gazebo>
-  <gazebo reference="front_left_wheel_link">
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
File: src/auto_vehicle/urdf/vehicle.xacro (robot description, xacro)
@@ -487,4 +487,6 @@
       <visualize>true</visualize>
       <topic>camera</topic>
+      <pose>0 0 0 0 0 0</pose>
+      <always_on>true</always_on>
       <camera name="head">
         <horizontal_fov>${camera_fov}</horizontal_fov>
@@ -498,4 +500,12 @@
           <far>300</far>
         </clip>
+        <distortion>
+          <k1>0.0</k1>
+          <k2>0.0</k2>
+          <k3>0.0</k3>
+          <p1>0.0</p1>
+          <p2>0.0</p2>
+          <center>0.5 0.5</center>
+        </distortion>
         <noise>
           <type>gaussian</type>
@@ -504,16 +514,4 @@
         </noise>
       </camera>
-      <plugin name="camera_controller" filename="libgazebo_ros_camera.so">
-        <alwaysOn>true</alwaysOn>
-        <updateRate>0.0</updateRate>
-        <cameraName>vehicle_front_camera</cameraName>
-        <frameName>camera_link</frameName>
-        <hackBaseline>0.07</hackBaseline>
-        <distortionK1>0.0</distortionK1>
-        <distortionK2>0.0</distortionK2>
-        <distortionK3>0.0</distortionK3>
-        <distortionT1>0.0</distortionT1>
-        <distortionT2>0.0</distortionT2>
-      </plugin>
     </sensor>
   </gazebo>
