Commit message: Set camera back from the front edge to keep the front wheel in frame
Add a camera_setback parameter and mount the camera stick that far
behind the body's front edge, so the front wheel's steering angle is
visible in the feed instead of being just out of frame ahead of it.

Also drop the offset_m extrapolation to the vehicle's row: with the
camera pulled back, the visible lane can start well short of that row,
and extrapolating that gap with the near tangent would swing the offset
more than it corrects. Use the chain's near point directly instead.

Co-Authored-By: Claude Sonnet 5 <noreply@anthropic.com>

File: src/auto_vehicle/urdf/vehicle.xacro (robot description, xacro)
@@ -18,4 +18,5 @@
   <xacro:arg name="camera_height" default="1.5" />
   <xacro:arg name="camera_pitch" default="0.1" />
+  <xacro:arg name="camera_setback" default="0.3" />
   <xacro:arg name="camera_fov" default="1.396263" />
   <xacro:arg name="camera_fps" default="30" />
@@ -41,4 +42,5 @@
   <xacro:property name="camera_height" value="$(arg camera_height)"/>
   <xacro:property name="camera_pitch" value="$(arg camera_pitch)"/>
+  <xacro:property name="camera_setback" value="$(arg camera_setback)"/>
   <xacro:property name="camera_fov" value="$(arg camera_fov)"/>
   <xacro:property name="camera_fps" value="$(arg camera_fps)"/>
@@ -378,5 +380,5 @@
   <joint name="camera_stick_joint" type="fixed">
     <axis xyz="0 1 0" />
-    <origin xyz="${body_length/2 - camera_stick_size/2} ${camera_box_size/2 + camera_stick_size/2} ${camera_height/2}" rpy="0.0 0.0 0.0"/>
+    <origin xyz="${body_length/2 - camera_stick_size/2 - camera_setback} ${camera_box_size/2 + camera_stick_size/2} ${camera_height/2}" rpy="0.0 0.0 0.0"/>
     <parent link="body_link"/>
     <child link="camera_stick_link"/>
