Commit message: Remove STM32 ros2_control interface, switch real vehicle to hyper_interface Arduino bridge
Also resolves the previous merge (9cb26d7) properly -- that commit had
unresolved <<<<<<< conflict markers left literally inside
real.launch.py, breaking it. Drops the STM32 SystemInterface plugin
(headers, source, build wiring, xacro ros2_control block) and the
STM32-only single_output mode on vehicle_controller_node; real.launch.py
and phone_control_real.launch.py now wire up hyper_interface's
arduino_interface_node instead, which subscribes to /velocity and
/steering_angle directly.

Co-Authored-By: Claude Sonnet 5 <noreply@anthropic.com>

File: src/control/hyper_control/urdf/vehicle.xacro (robot description, xacro)
@@ -3,6 +3,4 @@
   <!-- Arguments -->
   <xacro:arg name="use_sim" default="true" />
-  <xacro:arg name="serial_port" default="/dev/stm32" />
-  <xacro:arg name="baud_rate" default="115200" />
   <xacro:arg name="body_length" default="2.0" />
   <xacro:arg name="body_width" default="1.0" />
@@ -494,28 +492,4 @@
     </ros2_control>
   </xacro:if>
-  <!-- Real Vehicle Control (STM32) -->
-  <xacro:unless value="$(arg use_sim)">
-    <ros2_control name="control" type="system">
-      <hardware>
-        <plugin>hyper_control/Stm32SystemInterface</plugin>
-        <param name="serial_port">$(arg serial_port)</param>
-        <param name="baud_rate">$(arg baud_rate)</param>
-      </hardware>
-      <joint name="steering_joint">
-        <command_interface name="position">
-          <param name="min">${-max_steering_angle}</param>
-          <param name="max">${max_steering_angle}</param>
-        </command_interface>
-        <state_interface name="position"/>
-      </joint>
-      <joint name="rear_axle_joint">
-        <command_interface name="velocity">
-          <param name="min">${-max_wheel_angular_velocity}</param>
-          <param name="max">${max_wheel_angular_velocity}</param>
-        </command_interface>
-        <state_interface name="velocity"/>
-      </joint>
-    </ros2_control>
-  </xacro:unless>
   <!-- Gazebo Plugins -->
   <gazebo>

Commit message: feat: GPS heading 보정률 개선, GUI 웨이포인트 녹화, 수동/미션 launch 분리
이번 세션 작업:

gps_heading
- /gps/fix 차분을 슬라이딩 윈도우로 변경. 기존에는 거리 조건 미달로 기각할
  때도 _last_fix를 옮겨 기선이 항상 fix 한 칸에 묶였고, 그 결과 코스 보정이
  0.83Hz까지 떨어졌다. 이제 min_fix_displacement 이상 떨어진 가장 최근 fix와
  짝지어 fix rate 그대로(측정 4.1Hz) 코스가 나온다.
- max_baseline_age(3초) 추가. 정지/fix 유실 시 창을 비워 기선이 제자리
  회전을 가로지르지 않게 한다.
- 위 수정으로 odometry.launch.py의 sim 전용 min_fix_displacement 임시
  오버라이드를 제거했다. fix_position_stddev는 sim GPS 노이즈(~1cm) 기준으로
  유지한다.

웨이포인트 녹화
- waypoint_recorder_node에 ~/start, ~/stop 서비스와 auto_start 파라미터 추가.
  파일 열기를 생성자에서 start_recording으로 옮겨, 노드가 떠 있는 것과 기록
  중인 것을 분리했다 -- 스택을 띄우는 것만으로 지난 녹화본이 truncate되지
  않는다. auto_start 기본값은 true라 기존 ros2 run 사용법은 그대로다.
- ~/status(String), ~/path(Path)를 transient_local로 발행.
- waypoint_record_gui.py 추가. Record/Stop 버튼, 점 수/누적 거리/다음 점까지
  남은 거리/GPS 상태/EKF 공분산과 찍힌 점 미니맵을 실시간 표시한다.
- record.launch.py로 레코더+GUI를 묶어 수동 주행 launch 양쪽에서 include.

launch 분리
- joystick_control_real.launch.py 신규. 수동 주행 전용이며 perception을 띄우지
  않고 녹화 스택을 포함한다.
- real.launch.py에서 use_joystick 제거. joystick_controller_node와
  cmd_vel_to_ackermann_node가 /velocity, /steering_angle을 동시에 100Hz로 쏘는
  사고를 인자 하나로 낼 수 있었다. 이제 미션 전용이다.
- real.launch.py에 waypoint_csv 인자를 선언하고 behavior 스테이지로 전달.
  기존에는 인자를 줘도 조용히 무시되어 실차에 sim.csv가 실렸다.
- phone_control_real.launch.py에도 녹화 스택 추가.

mission_loader
- 라벨 값 'last'를 CSV 마지막 웨이포인트 센티널로 허용. simple.yaml의
  course_end가 sim.csv 좌표라 real.csv로는 스냅 허용치를 넘겨 로드가 거부되던
  문제를 없앤다. 좌표 라벨 경로는 그대로다(mission.yaml 17스텝 로드 확인).

문서
- hyper_launch/AUG30.md 신규(실차 테스트 절차), hyper_waypoint/README.md,
  hyper_launch/README.md 갱신.

이 커밋에는 브랜치에 남아 있던 진행 중 작업(hyper_lane_detection,
hyper_camera, hyper_control, hyper_gazebo, hyper_object_detection 등)도 함께
포함된다.

Co-Authored-By: Claude Opus 5 <noreply@anthropic.com>

File: src/control/hyper_control/urdf/vehicle.xacro (robot description, xacro)
@@ -27,20 +27,4 @@
   <xacro:arg name="object_camera_setback" default="0.5" />
   <xacro:arg name="object_camera_fov" default="1.2217305" />
-  <!-- Rear camera: RGBD, modelled on the Intel RealSense D435i the real car already carries
-       (see hyper_launch/sensors.launch.py, where it currently supplies /imu only). Gazebo's
-       rgbd_camera renders colour and depth through one shared lens, so the single
-       horizontal_fov below is the D435i's *depth* FOV (87 deg), not its narrower RGB FOV
-       (69 deg); depth is why this sensor is RGBD at all. rear_image_* are pixels, the other
-       rear_camera_* are the mounting pose, kept separate from the front camera's so the rear's
-       geometry no longer moves whenever the front fisheye is retuned. -->
-  <xacro:arg name="rear_camera_height" default="0.3" />
-  <xacro:arg name="rear_camera_pitch" default="0.0" />
-  <xacro:arg name="rear_camera_setback" default="0.0" />
-  <xacro:arg name="rear_camera_fov" default="1.5184364" />
-  <xacro:arg name="rear_camera_fps" default="30" />
-  <xacro:arg name="rear_image_width" default="848" />
-  <xacro:arg name="rear_image_height" default="480" />
-  <xacro:arg name="rear_depth_near" default="0.2" />
-  <xacro:arg name="rear_depth_far" default="10.0" />
   <!-- Mathematical Constants -->
   <xacro:property name="PI" value="3.14159265"/>
@@ -70,13 +54,4 @@
   <xacro:property name="object_camera_setback" value="$(arg object_camera_setback)"/>
   <xacro:property name="object_camera_fov" value="$(arg object_camera_fov)"/>
-  <xacro:property name="rear_camera_height" value="$(arg rear_camera_height)"/>
-  <xacro:property name="rear_camera_pitch" value="$(arg rear_camera_pitch)"/>
-  <xacro:property name="rear_camera_setback" value="$(arg rear_camera_setback)"/>
-  <xacro:property name="rear_camera_fov" value="$(arg rear_camera_fov)"/>
-  <xacro:property name="rear_camera_fps" value="$(arg rear_camera_fps)"/>
-  <xacro:property name="rear_image_width" value="$(arg rear_image_width)"/>
-  <xacro:property name="rear_image_height" value="$(arg rear_image_height)"/>
-  <xacro:property name="rear_depth_near" value="$(arg rear_depth_near)"/>
-  <xacro:property name="rear_depth_far" value="$(arg rear_depth_far)"/>
   <xacro:property name="body_mass" value="${body_density * body_length * body_height * body_width}"/>
   <xacro:property name="body_inertia_x" value="${1.0/12.0 * body_mass * (body_height*body_height + body_width*body_width)}"/>
@@ -289,27 +264,4 @@
       </geometry>
       <material name="object_camera_material">
-        <color rgba="0.0 0.0 0.0 1.0"/>
-      </material>
-    </visual>
-    <inertial>
-      <mass value="1e-5" />
-      <origin xyz="0 0 0" rpy="0 0 0"/>
-      <inertia ixx="1e-6" ixy="0" ixz="0" iyy="1e-6" iyz="0" izz="1e-6" />
-    </inertial>
-  </link>
-  <!-- Rear Camera Link -->
-  <link name="rear_camera_link">
-    <collision>
-      <origin xyz="0 0 0" rpy="0 0 0"/>
-      <geometry>
-        <box size="${camera_box_size} ${camera_box_size} ${camera_box_size}"/>
-      </geometry>
-    </collision>
-    <visual>
-      <origin xyz="0 0 0" rpy="0 0 0"/>
-      <geometry>
-        <box size="${camera_box_size} ${camera_box_size} ${camera_box_size}"/>
-      </geometry>
-      <material name="rear_camera_material">
         <color rgba="0.0 0.0 0.0 1.0"/>
       </material>
@@ -455,11 +407,4 @@
     <parent link="body_link"/>
     <child link="object_camera_link"/>
-  </joint>
-  <!-- Rear Camera Joint -->
-  <joint name="rear_camera_joint" type="fixed">
-    <axis xyz="0 1 0" />
-    <origin xyz="${-(body_length/2 - camera_box_size/2 - rear_camera_setback)} 0.0 ${rear_camera_height}" rpy="0 ${rear_camera_pitch} ${PI}"/>
-    <parent link="body_link"/>
-    <child link="rear_camera_link"/>
   </joint>
   <gazebo reference="body_link">
@@ -607,67 +552,4 @@
     </sensor>
   </gazebo>
-  <!-- Rear Camera (RGBD, Intel RealSense D435i-equivalent) -->
-  <!-- Publishes four ign topics off <topic>: camera_rear/image (colour),
-       camera_rear/depth_image, camera_rear/points and camera_rear/camera_info. All four are
-       bridged in hyper_gazebo's ros_gz_bridge.yaml; the colour one keeps the ROS name
-       /camera_rear/image_raw its existing subscribers already use.
-       Spec source: Intel RealSense D435i datasheet:
-         depth FOV      87 x 58 deg  -> horizontal_fov 1.5184364 rad, and 848x480 is the D435i
-                                       depth mode whose aspect ratio reproduces ~58 deg vertically
-                                       (2*atan(tan(43.5 deg) * 480/848) = 56.5 deg)
-         depth range    ~0.2 m min-Z to ~10 m -> <depth_camera><clip>
-         frame rate     30 Hz (the D435i also does 90 Hz at this resolution; 30 keeps the sim's
-                        software-rendered (LIBGL_ALWAYS_SOFTWARE=1) render budget sane)
-       The colour <clip> deliberately stays at the wide render range rather than the depth
-       range; the D435i's RGB stream is an ordinary camera that sees past 10 m; only its
-       depth is limited. Gazebo shares one lens between the two streams, so the colour image
-       comes out at the 87 deg depth FOV rather than the D435i's 69 deg RGB FOV (see the args
-       block for why depth wins that trade).
-       The libgazebo_ros_camera.so plugin the old <sensor> carried was Gazebo Classic config
-       and was inert under ign-gazebo, so it is not carried over. -->
-  <gazebo reference="rear_camera_link">
-    <sensor type="rgbd_camera" name="vehicle_rear_camera">
-      <update_rate>${rear_camera_fps}</update_rate>
-      <visualize>true</visualize>
-      <topic>camera_rear</topic>
-      <!-- All four streams are stamped with this frame. Deliberately rear_camera_link (REP-103
-           body convention, x forward) and NOT a z-forward optical frame: ign-sensors emits the
-           point cloud's xyz in the camera link's own convention, x = range, so the measured
-           cloud only lines up with TF if the frame it names is the x-forward one. sdformat's
-           <optical_frame_id> is a label only here; it renames the frame without rotating the
-           data, which would silently tip the cloud 90 deg. Anyone adding depth_image_proc
-           later does need a z-forward frame for /camera_rear/depth/image_raw + camera_info,
-           and should publish that frame explicitly rather than relabelling this sensor.
-           depthimage_to_laserscan (see hyper_object_detection's perception.launch.py) is NOT
-           such a consumer: it reads the depth image's *pixels*, never its frame_id, and names
-           its output frame through the output_frame parameter, which is this link because
-           a LaserScan's own convention (x along the view direction, y to its left) is exactly
-           this link's, not an optical frame's. -->
-      <gz_frame_id>rear_camera_link</gz_frame_id>
-      <camera name="rear">
-        <horizontal_fov>${rear_camera_fov}</horizontal_fov>
-        <image>
-          <width>${rear_image_width}</width>
-          <height>${rear_image_height}</height>
-          <format>R8G8B8</format>
-        </image>
-        <clip>
-          <near>0.02</near>
-          <far>550</far>
-        </clip>
-        <depth_camera>
-          <clip>
-            <near>${rear_depth_near}</near>
-            <far>${rear_depth_far}</far>
-          </clip>
-        </depth_camera>
-        <noise>
-          <type>gaussian</type>
-          <mean>0.0</mean>
-          <stddev>0.007</stddev>
-        </noise>
-      </camera>
-    </sensor>
-  </gazebo>
   <!-- IMU sensor -->
   <gazebo reference="body_link">
@@ -756,6 +638,8 @@
                arc does not sharpen the sensor, so the sample count has to halve with it.
                Consequence, deliberately: nothing raytrace-clears the rear of the local costmap
-               except the rear camera's /scan_rear, whose FOV is 87 deg. See the scan and
-               rear_scan blocks in hyper_planner/config/nav2_controller.yaml. -->
+               at all, now that the rear camera (and with it /scan_rear) is gone. Cells marked
+               while driving forward survive behind the vehicle until the costmap's rolling
+               window drops them. See the scan block in
+               hyper_planner/config/nav2_controller.yaml. -->
           <horizontal>
             <samples>360</samples>
