Commit message: feat: Implement STM32 system interface for vehicle control and update URDF configuration

File: src/control/hyper_control/urdf/vehicle.xacro (robot description, xacro)
@@ -2,4 +2,7 @@
 <robot name="ackermann_steering_vehicle" xmlns:xacro="http://www.ros.org/wiki/xacro">
   <!-- Arguments -->
+  <xacro:arg name="use_sim" default="true" />
+  <xacro:arg name="serial_port" default="/dev/ttyUSB0" />
+  <xacro:arg name="baud_rate" default="115200" />
   <xacro:arg name="body_length" default="2.0" />
   <xacro:arg name="body_width" default="1.0" />
@@ -448,45 +451,71 @@
   </gazebo>
   <!-- Gazebo Control -->
-  <ros2_control name="control" type="system">
-    <hardware>
-      <plugin>gz_ros2_control/GazeboSimSystem</plugin>
-    </hardware>
-    <joint name="front_left_steering_joint">
-      <command_interface name="position">
-        <param name="min">${-max_steering_angle}</param>
-        <param name="max">${max_steering_angle}</param>
-      </command_interface>
-      <state_interface name="position"/>
-      <state_interface name="velocity"/>
-      <state_interface name="effort"/>
-    </joint>
-    <joint name="front_right_steering_joint">
-      <command_interface name="position">
-        <param name="min">${-max_steering_angle}</param>
-        <param name="max">${max_steering_angle}</param>
-      </command_interface>
-      <state_interface name="position"/>
-      <state_interface name="velocity"/>
-      <state_interface name="effort"/>
-    </joint>
-    <joint name="rear_left_wheel_joint">
-      <command_interface name="velocity">
-        <param name="min">${-max_wheel_angular_velocity}</param>
-        <param name="max">${max_wheel_angular_velocity}</param>
-      </command_interface>
-      <state_interface name="position"/>
-      <state_interface name="velocity"/>
-      <state_interface name="effort"/>
-    </joint>
-    <joint name="rear_right_wheel_joint">
-      <command_interface name="velocity">
-        <param name="min">${-max_wheel_angular_velocity}</param>
-        <param name="max">${max_wheel_angular_velocity}</param>
-      </command_interface>
-      <state_interface name="position"/>
-      <state_interface name="velocity"/>
-      <state_interface name="effort"/>
-    </joint>
-  </ros2_control>
+  <xacro:if value="$(arg use_sim)">
+    <ros2_control name="control" type="system">
+      <hardware>
+        <plugin>gz_ros2_control/GazeboSimSystem</plugin>
+      </hardware>
+      <joint name="front_left_steering_joint">
+        <command_interface name="position">
+          <param name="min">${-max_steering_angle}</param>
+          <param name="max">${max_steering_angle}</param>
+        </command_interface>
+        <state_interface name="position"/>
+        <state_interface name="velocity"/>
+        <state_interface name="effort"/>
+      </joint>
+      <joint name="front_right_steering_joint">
+        <command_interface name="position">
+          <param name="min">${-max_steering_angle}</param>
+          <param name="max">${max_steering_angle}</param>
+        </command_interface>
+        <state_interface name="position"/>
+        <state_interface name="velocity"/>
+        <state_interface name="effort"/>
+      </joint>
+      <joint name="rear_left_wheel_joint">
+        <command_interface name="velocity">
+          <param name="min">${-max_wheel_angular_velocity}</param>
+          <param name="max">${max_wheel_angular_velocity}</param>
+        </command_interface>
+        <state_interface name="position"/>
+        <state_interface name="velocity"/>
+        <state_interface name="effort"/>
+      </joint>
+      <joint name="rear_right_wheel_joint">
+        <command_interface name="velocity">
+          <param name="min">${-max_wheel_angular_velocity}</param>
+          <param name="max">${max_wheel_angular_velocity}</param>
+        </command_interface>
+        <state_interface name="position"/>
+        <state_interface name="velocity"/>
+        <state_interface name="effort"/>
+      </joint>
+    </ros2_control>
+  </xacro:if>
+  <!-- Real Vehicle Control (STM32) -->
+  <xacro:unless value="$(arg use_sim)">
+    <ros2_control name="control" type="system">
+      <hardware>
+        <plugin>hyper_control/Stm32SystemInterface</plugin>
+        <param name="serial_port">$(arg serial_port)</param>
+        <param name="baud_rate">$(arg baud_rate)</param>
+      </hardware>
+      <joint name="steering_joint">
+        <command_interface name="position">
+          <param name="min">${-max_steering_angle}</param>
+          <param name="max">${max_steering_angle}</param>
+        </command_interface>
+        <state_interface name="position"/>
+      </joint>
+      <joint name="rear_axle_joint">
+        <command_interface name="velocity">
+          <param name="min">${-max_wheel_angular_velocity}</param>
+          <param name="max">${max_wheel_angular_velocity}</param>
+        </command_interface>
+        <state_interface name="velocity"/>
+      </joint>
+    </ros2_control>
+  </xacro:unless>
   <!-- Gazebo Plugins -->
   <gazebo>

Commit message: Refactor mission manager node and update ROS-GZ bridge configuration
- Removed unused includes and restructured code in mission_manager_node.cpp for better readability and maintainability.
- Integrated mission loading functionality into a separate MissionLoader class to streamline mission loading process.
- Updated the waypoints and steps handling to utilize the new MissionLoader.
- Enhanced the PathProgress class to manage progress tracking more effectively.
- Added new camera topics for the rear RGBD camera in ros_gz_bridge.yaml to support depth image and point cloud data.
- Adjusted existing camera topic configurations to align with the new structure.

File: src/control/hyper_control/urdf/vehicle.xacro (robot description, xacro)
@@ -29,4 +29,20 @@
   <xacro:arg name="object_camera_setback" default="0.5" />
   <xacro:arg name="object_camera_fov" default="1.2217305" />
+  <!-- Rear camera: RGBD, modelled on the Intel RealSense D435i the real car already carries
+       (see hyper_launch/sensors.launch.py, where it currently supplies /imu only). Gazebo's
+       rgbd_camera renders colour and depth through one shared lens, so the single
+       horizontal_fov below is the D435i's *depth* FOV (87 deg), not its narrower RGB FOV
+       (69 deg); depth is why this sensor is RGBD at all. rear_image_* are pixels, the other
+       rear_camera_* are the mounting pose, kept separate from the front camera's so the rear's
+       geometry no longer moves whenever the front fisheye is retuned. -->
+  <xacro:arg name="rear_camera_height" default="1.5" />
+  <xacro:arg name="rear_camera_pitch" default="0.1" />
+  <xacro:arg name="rear_camera_setback" default="0.3" />
+  <xacro:arg name="rear_camera_fov" default="1.5184364" />
+  <xacro:arg name="rear_camera_fps" default="30" />
+  <xacro:arg name="rear_image_width" default="848" />
+  <xacro:arg name="rear_image_height" default="480" />
+  <xacro:arg name="rear_depth_near" default="0.2" />
+  <xacro:arg name="rear_depth_far" default="10.0" />
   <!-- Mathematical Constants -->
   <xacro:property name="PI" value="3.14159265"/>
@@ -56,4 +72,13 @@
   <xacro:property name="object_camera_setback" value="$(arg object_camera_setback)"/>
   <xacro:property name="object_camera_fov" value="$(arg object_camera_fov)"/>
+  <xacro:property name="rear_camera_height" value="$(arg rear_camera_height)"/>
+  <xacro:property name="rear_camera_pitch" value="$(arg rear_camera_pitch)"/>
+  <xacro:property name="rear_camera_setback" value="$(arg rear_camera_setback)"/>
+  <xacro:property name="rear_camera_fov" value="$(arg rear_camera_fov)"/>
+  <xacro:property name="rear_camera_fps" value="$(arg rear_camera_fps)"/>
+  <xacro:property name="rear_image_width" value="$(arg rear_image_width)"/>
+  <xacro:property name="rear_image_height" value="$(arg rear_image_height)"/>
+  <xacro:property name="rear_depth_near" value="$(arg rear_depth_near)"/>
+  <xacro:property name="rear_depth_far" value="$(arg rear_depth_far)"/>
   <xacro:property name="body_mass" value="${body_density * body_length * body_height * body_width}"/>
   <xacro:property name="body_inertia_x" value="${1.0/12.0 * body_mass * (body_height*body_height + body_width*body_width)}"/>
@@ -426,5 +451,5 @@
   <joint name="rear_camera_joint" type="fixed">
     <axis xyz="0 1 0" />
-    <origin xyz="${-(body_length/2 - camera_box_size/2 - camera_setback)} 0.0 ${camera_height}" rpy="0 ${camera_pitch} ${PI}"/>
+    <origin xyz="${-(body_length/2 - camera_box_size/2 - rear_camera_setback)} 0.0 ${rear_camera_height}" rpy="0 ${rear_camera_pitch} ${PI}"/>
     <parent link="body_link"/>
     <child link="rear_camera_link"/>
@@ -613,15 +638,42 @@
     </sensor>
   </gazebo>
-  <!-- Rear Camera -->
+  <!-- Rear Camera (RGBD, Intel RealSense D435i-equivalent) -->
+  <!-- Publishes four ign topics off <topic>: camera_rear/image (colour),
+       camera_rear/depth_image, camera_rear/points and camera_rear/camera_info. All four are
+       bridged in hyper_gazebo's ros_gz_bridge.yaml; the colour one keeps the ROS name
+       /camera_rear/image_raw its existing subscribers already use.
+       Spec source: Intel RealSense D435i datasheet:
+         depth FOV      87 x 58 deg  -> horizontal_fov 1.5184364 rad, and 848x480 is the D435i
+                                       depth mode whose aspect ratio reproduces ~58 deg vertically
+                                       (2*atan(tan(43.5 deg) * 480/848) = 56.5 deg)
+         depth range    ~0.2 m min-Z to ~10 m -> <depth_camera><clip>
+         frame rate     30 Hz (the D435i also does 90 Hz at this resolution; 30 keeps the sim's
+                        software-rendered (LIBGL_ALWAYS_SOFTWARE=1) render budget sane)
+       The colour <clip> deliberately stays at the wide render range rather than the depth
+       range; the D435i's RGB stream is an ordinary camera that sees past 10 m; only its
+       depth is limited. Gazebo shares one lens between the two streams, so the colour image
+       comes out at the 87 deg depth FOV rather than the D435i's 69 deg RGB FOV (see the args
+       block for why depth wins that trade).
+       The libgazebo_ros_camera.so plugin the old <sensor> carried was Gazebo Classic config
+       and was inert under ign-gazebo, so it is not carried over. -->
   <gazebo reference="rear_camera_link">
-    <sensor type="camera" name="vehicle_rear_camera">
-      <update_rate>${camera_fps}</update_rate>
+    <sensor type="rgbd_camera" name="vehicle_rear_camera">
+      <update_rate>${rear_camera_fps}</update_rate>
       <visualize>true</visualize>
       <topic>camera_rear</topic>
+      <!-- All four streams are stamped with this frame. Deliberately rear_camera_link (REP-103
+           body convention, x forward) and NOT a z-forward optical frame: ign-sensors emits the
+           point cloud's xyz in the camera link's own convention, x = range, so the measured
+           cloud only lines up with TF if the frame it names is the x-forward one. sdformat's
+           <optical_frame_id> is a label only here; it renames the frame without rotating the
+           data, which would silently tip the cloud 90 deg. Anyone adding depth_image_proc
+           later does need a z-forward frame for /camera_rear/depth/image_raw + camera_info,
+           and should publish that frame explicitly rather than relabelling this sensor. -->
+      <gz_frame_id>rear_camera_link</gz_frame_id>
       <camera name="rear">
-        <horizontal_fov>${camera_fov}</horizontal_fov>
+        <horizontal_fov>${rear_camera_fov}</horizontal_fov>
         <image>
-          <width>${image_width}</width>
-          <height>${image_height}</height>
+          <width>${rear_image_width}</width>
+          <height>${rear_image_height}</height>
           <format>R8G8B8</format>
         </image>
@@ -630,4 +682,10 @@
           <far>550</far>
         </clip>
+        <depth_camera>
+          <clip>
+            <near>${rear_depth_near}</near>
+            <far>${rear_depth_far}</far>
+          </clip>
+        </depth_camera>
         <noise>
           <type>gaussian</type>
@@ -636,16 +694,4 @@
         </noise>
       </camera>
-      <plugin name="rear_camera_controller" filename="libgazebo_ros_camera.so">
-        <alwaysOn>true</alwaysOn>
-        <updateRate>0.0</updateRate>
-        <cameraName>vehicle_rear_camera</cameraName>
-        <frameName>rear_camera_link</frameName>
-        <hackBaseline>0.07</hackBaseline>
-        <distortionK1>0.0</distortionK1>
-        <distortionK2>0.0</distortionK2>
-        <distortionK3>0.0</distortionK3>
-        <distortionT1>0.0</distortionT1>
-        <distortionT2>0.0</distortionT2>
-      </plugin>
     </sensor>
   </gazebo>

Commit message: Add SUV model and update track world with new obstacles
- Created model configuration (model.config) and SDF file (model.sdf) for a new SUV model.
- Updated the track world to include the new SUV model and additional obstacles, including a pedestrian and parked vehicles along the acceleration path.
- Adjusted physics parameters for improved simulation performance.

File: src/control/hyper_control/urdf/vehicle.xacro (robot description, xacro)
@@ -372,6 +372,16 @@
   </joint>
 <!-- LiDAR Fixed Joint -->
+  <!-- 스캔 평면 높이 = wheel_radius*1.5 + body_height/2 + 이 오프셋
+       = 0.30 + 0.20 + 0.15 = 지면 위 0.65 m (parameters.yaml 기준값).
+       0.25 -> 0.15으로 10 cm 낮췄습니다. 이유:
+         - 이전 높이(0.75 m)는 hatchback 장애물 지붕(0.778 m)의 위쪽 2.8 cm를 스치기만 해서,
+           피치에 따라 반사가 들어왔다 말았다 했습니다(= local costmap이 비어 MPPI가 직진).
+           0.65 m면 지붕보다 12.8 cm 아래라 차체를 확실히 때립니다.
+         - 아래로는 차체 박스 윗면(0.50 m)보다 15 cm 위여야 gpu_lidar가 자기 차체에
+           가리지 않습니다.
+       주의: 이 xacro는 real.launch.py도 같이 씁니다. 실차 라이다를 실제로 0.65 m로
+       내려 달지 않으면 body_link->lidar_link TF가 실측과 어긋납니다. -->
   <joint name="lidar_joint" type="fixed">
-    <origin xyz="0.15 0 ${body_height/2 + 0.25}" rpy="0 0 0"/>
+    <origin xyz="0.15 0 ${body_height/2 + 0.15}" rpy="0 0 0"/>
     <parent link="body_link"/>
     <child link="lidar_link"/>
@@ -544,4 +554,10 @@
       <visualize>true</visualize>
       <topic>camera</topic>
+      <!-- ign publishes the image on <topic> and its camera_info on <topic>_info; both are
+           bridged in hyper_gazebo's ros_gz_bridge.yaml (camera -> /camera/image_raw,
+           camera_info -> /camera/info). The libgazebo_ros_camera.so plugin this sensor used
+           to carry was Gazebo Classic config, inert under ign-gazebo, so it is not carried
+           over; its frameName is what the gz_frame_id below replaces. -->
+      <gz_frame_id>camera_link</gz_frame_id>
       <camera name="head">
         <horizontal_fov>${camera_fov}</horizontal_fov>
@@ -561,16 +577,4 @@
         </noise>
       </camera>
-      <plugin name="camera_controller" filename="libgazebo_ros_camera.so">
-        <alwaysOn>true</alwaysOn>
-        <updateRate>0.0</updateRate>
-        <cameraName>vehicle_front_camera</cameraName>
-        <frameName>camera_link</frameName>
-        <hackBaseline>0.07</hackBaseline>
-        <distortionK1>0.0</distortionK1>
-        <distortionK2>0.0</distortionK2>
-        <distortionK3>0.0</distortionK3>
-        <distortionT1>0.0</distortionT1>
-        <distortionT2>0.0</distortionT2>
-      </plugin>
     </sensor>
   </gazebo>
@@ -581,4 +585,7 @@
       <visualize>true</visualize>
       <topic>camera_object</topic>
+      <!-- Bridged as camera_object -> /camera_object/image_raw and camera_object_info ->
+           /camera_object/info. Same Classic-plugin removal as the front camera above. -->
+      <gz_frame_id>object_camera_link</gz_frame_id>
       <camera name="object">
         <horizontal_fov>${object_camera_fov}</horizontal_fov>
@@ -598,16 +605,4 @@
         </noise>
       </camera>
-      <plugin name="object_camera_controller" filename="libgazebo_ros_camera.so">
-        <alwaysOn>true</alwaysOn>
-        <updateRate>0.0</updateRate>
-        <cameraName>vehicle_object_camera</cameraName>
-        <frameName>object_camera_link</frameName>
-        <hackBaseline>0.07</hackBaseline>
-        <distortionK1>0.0</distortionK1>
-        <distortionK2>0.0</distortionK2>
-        <distortionK3>0.0</distortionK3>
-        <distortionT1>0.0</distortionT1>
-        <distortionT2>0.0</distortionT2>
-      </plugin>
     </sensor>
   </gazebo>

Commit message: Update measure

File: src/control/hyper_control/urdf/vehicle.xacro (robot description, xacro)
@@ -318,6 +318,13 @@
   </link>
 <!-- GPS Fixed Joint -->
+  <!-- 실측(2026-08-30): 안테나가 body_link 중심에서 뒤로 0.23 m, 좌우 중앙, 지면 위 1.118 m
+       (라이드 하이트 0.171 m을 빼면 body_link 기준 0.947 m). body_height 수식 대신 리터럴로
+       박아 넣었습니다 -- body_height 자체가 아직 실측 전(placeholder 0.40)이라 수식으로는
+       실측치를 정확히 못 담습니다. gps_link는 시각화(RViz)용일 뿐 navsat_transform 등
+       어떤 로컬라이제이션 코드도 이 TF를 안 씁니다(안테나 레버암 보정이 없음) -- 그래도
+       실측치를 넣어 두는 이유는 나중에 레버암 보정을 추가하게 되거나 시각화 정확도가
+       필요해질 때를 위해서입니다. -->
   <joint name="gps_joint" type="fixed">
-    <origin xyz="0 0 ${body_height/2 + 0.25}" rpy="0 0 0"/>
+    <origin xyz="-0.23 0 0.947" rpy="0 0 0"/>
     <parent link="body_link"/>
     <child link="gps_link"/>

Commit message: feat: add wheel_base parameter and update related configurations

File: src/control/hyper_control/urdf/vehicle.xacro (robot description, xacro)
@@ -7,4 +7,5 @@
   <xacro:arg name="body_height" default="0.5" />
   <xacro:arg name="body_density" default="1000.0" />
+  <xacro:arg name="wheel_base" default="1.4" />
   <xacro:arg name="wheel_radius" default="0.3" />
   <xacro:arg name="wheel_width" default="0.1" />
@@ -34,4 +35,5 @@
   <xacro:property name="body_height" value="$(arg body_height)"/>
   <xacro:property name="body_density" value="$(arg body_density)"/>
+  <xacro:property name="wheel_base" value="$(arg wheel_base)"/>
   <xacro:property name="wheel_radius" value="$(arg wheel_radius)"/>
   <xacro:property name="wheel_width" value="$(arg wheel_width)"/>
@@ -59,5 +61,7 @@
   <xacro:property name="body_inertia_z" value="${1.0/12.0 * body_mass * (body_length*body_length + body_width*body_width)}"/>
   <xacro:property name="wheel_separation" value="${body_width + wheel_width}"/>
-  <xacro:property name="wheel_offset" value="${body_length/2 - wheel_radius}"/>
+  <!-- Front/rear axle half-spacing. Driven by the measured wheel_base, NOT body_length,
+       so the sim Ackermann kinematics match the real vehicle (wheel_base != body_length). -->
+  <xacro:property name="wheel_offset" value="${wheel_base/2}"/>
   <xacro:property name="wheel_mass" value="${wheel_density * PI * wheel_radius * wheel_radius * wheel_width}"/>
   <xacro:property name="wheel_inertia_x" value="${1.0/12.0 * wheel_mass * (3*wheel_radius*wheel_radius + wheel_width*wheel_width)}"/>
