Commit message: Only one camera now, instead of two.

File: src/control/hyper_control/urdf/vehicle.xacro (robot description, xacro)
@@ -24,8 +24,4 @@
   <xacro:arg name="image_width" default="640" />
   <xacro:arg name="image_height" default="480" />
-  <xacro:arg name="object_camera_height" default="1.2" />
-  <xacro:arg name="object_camera_pitch" default="0.0" />
-  <xacro:arg name="object_camera_setback" default="0.5" />
-  <xacro:arg name="object_camera_fov" default="1.2217305" />
   <!-- Mathematical Constants -->
   <xacro:property name="PI" value="3.14159265"/>
@@ -52,8 +48,4 @@
   <xacro:property name="image_width" value="$(arg image_width)"/>
   <xacro:property name="image_height" value="$(arg image_height)"/>
-  <xacro:property name="object_camera_height" value="$(arg object_camera_height)"/>
-  <xacro:property name="object_camera_pitch" value="$(arg object_camera_pitch)"/>
-  <xacro:property name="object_camera_setback" value="$(arg object_camera_setback)"/>
-  <xacro:property name="object_camera_fov" value="$(arg object_camera_fov)"/>
   <xacro:property name="body_mass" value="${body_density * body_length * body_height * body_width}"/>
   <xacro:property name="body_inertia_x" value="${1.0/12.0 * body_mass * (body_height*body_height + body_width*body_width)}"/>
@@ -231,5 +223,9 @@
     </inertial>
   </link>
-  <!-- Camera Link -->
+  <!-- Camera Link. The vehicle's only camera: a Logitech C920 on the real car, feeding both
+       lane_detection (via a bird's-eye warp) and object_detection (YOLO). It replaced a pair of
+       cameras (a 153 deg ELP fisheye for lanes plus this C920 for objects), so its pose and FOV
+       below are the C920 mount's, and hyper_lane_detection's BEV had to give up the near field
+       for it. See kSimFrontNearM in lane_detection_node.cpp. -->
   <link name="camera_link">
     <collision>
@@ -245,27 +241,4 @@
       </geometry>
       <material name="camera_material">
-        <color rgba="0.0 0.0 0.0 1.0"/>
-      </material>
-    </visual>
-    <inertial>
-      <mass value="1e-5" />
-      <origin xyz="0 0 0" rpy="0 0 0"/>
-      <inertia ixx="1e-6" ixy="0" ixz="0" iyy="1e-6" iyz="0" izz="1e-6" />
-    </inertial>
-  </link>
-  <!-- Object Detection Camera Link (normal 70 deg hfov, front-facing) -->
-  <link name="object_camera_link">
-    <collision>
-      <origin xyz="0 0 0" rpy="0 0 0"/>
-      <geometry>
-        <box size="${camera_box_size} ${camera_box_size} ${camera_box_size}"/>
-      </geometry>
-    </collision>
-    <visual>
-      <origin xyz="0 0 0" rpy="0 0 0"/>
-      <geometry>
-        <box size="${camera_box_size} ${camera_box_size} ${camera_box_size}"/>
-      </geometry>
-      <material name="object_camera_material">
         <color rgba="0.0 0.0 0.0 1.0"/>
       </material>
@@ -411,11 +384,4 @@
     <parent link="body_link"/>
     <child link="camera_link"/>
-  </joint>
-  <!-- Object Detection Camera Joint -->
-  <joint name="object_camera_joint" type="fixed">
-    <axis xyz="0 1 0" />
-    <origin xyz="${body_length/2 - camera_box_size/2 - object_camera_setback} 0.0 ${object_camera_height}" rpy="0 ${object_camera_pitch} 0"/>
-    <parent link="body_link"/>
-    <child link="object_camera_link"/>
   </joint>
   <gazebo reference="body_link">
@@ -504,5 +470,5 @@
     </plugin>
   </gazebo>
-  <!-- Camera -->
+  <!-- Camera. Shared by lane_detection and object_detection; there is only one. -->
   <gazebo reference="camera_link">
     <sensor type="camera" name="vehicle_front_camera">
@@ -518,32 +484,4 @@
       <camera name="head">
         <horizontal_fov>${camera_fov}</horizontal_fov>
-        <image>
-          <width>${image_width}</width>
-          <height>${image_height}</height>
-          <format>R8G8B8</format>
-        </image>
-        <clip>
-          <near>0.02</near>
-          <far>550</far>
-        </clip>
-        <noise>
-          <type>gaussian</type>
-          <mean>0.0</mean>
-          <stddev>0.007</stddev>
-        </noise>
-      </camera>
-    </sensor>
-  </gazebo>
-  <!-- Object Detection Camera -->
-  <gazebo reference="object_camera_link">
-    <sensor type="camera" name="vehicle_object_camera">
-      <update_rate>${camera_fps}</update_rate>
-      <visualize>true</visualize>
-      <topic>camera_object</topic>
-      <!-- Bridged as camera_object -> /camera_object/image_raw and camera_object_info ->
-           /camera_object/info. Same Classic-plugin removal as the front camera above. -->
-      <gz_frame_id>object_camera_link</gz_frame_id>
-      <camera name="object">
-        <horizontal_fov>${object_camera_fov}</horizontal_fov>
         <image>
           <width>${image_width}</width>

Commit message: Merged two gui to one

File: src/control/hyper_control/urdf/vehicle.xacro (robot description, xacro)
@@ -298,12 +298,59 @@
        (라이드 하이트 0.171 m을 빼면 body_link 기준 0.947 m). body_height 수식 대신 리터럴로
        박아 넣었습니다 — body_height 자체가 아직 실측 전(placeholder 0.40)이라 수식으로는
-       실측치를 정확히 못 담습니다. gps_link는 시각화(RViz)용일 뿐 navsat_transform 등
-       어떤 로컬라이제이션 코드도 이 TF를 안 씁니다(안테나 레버암 보정이 없음) — 그래도
-       실측치를 넣어 두는 이유는 나중에 레버암 보정을 추가하게 되거나 시각화 정확도가
-       필요해질 때를 위해서입니다. -->
+       실측치를 정확히 못 담습니다.
+       (예전 주석: "gps_link는 시각화용일 뿐 아무도 안 쓴다" — 지금은 아닙니다.)
+       navsat_transform_node가 이 TF를 실제로 씁니다: /gps/fix(뒤쪽 base 안테나)의
+       frame_id가 gps_link이고, navsat이 body_link -> gps_link로 안테나 레버암을 빼서
+       GPS 위치를 차량 중심 기준으로 옮깁니다. 즉 여기 xyz를 바꾸면 글로벌 EKF가
+       내는 위치가 그만큼 통째로 움직입니다 — 실측 없이 건드리지 마세요. -->
   <joint name="gps_joint" type="fixed">
     <origin xyz="-0.23 0 0.947" rpy="0 0 0"/>
     <parent link="body_link"/>
     <child link="gps_link"/>
+  </joint>
+  <!-- rover(앞쪽) 안테나. base와 함께 moving-base RTK 헤딩을 만드는 두 번째 ZED-F9P다.
+       색만 다르게(초록) 해서 RViz에서 base와 구분되게 둔다. -->
+  <link name="gps_rover_link">
+    <visual>
+      <origin xyz="0 0 0" rpy="0 0 0"/>
+      <geometry>
+        <box size="0.08 0.08 0.03"/>
+      </geometry>
+      <material name="gps_rover_material">
+        <color rgba="0.0 0.8 0.2 1.0"/>
+      </material>
+    </visual>
+    <collision>
+      <origin xyz="0 0 0" rpy="0 0 0"/>
+      <geometry>
+        <box size="0.08 0.08 0.03"/>
+      </geometry>
+    </collision>
+    <inertial>
+      <mass value="0.05"/>
+      <origin xyz="0 0 0" rpy="0 0 0"/>
+      <inertia ixx="1e-5" ixy="0" ixz="0" iyy="1e-5" iyz="0" izz="1e-5"/>
+    </inertial>
+  </link>
+<!-- GPS Rover Fixed Joint -->
+  <!-- x = -0.23 + 0.60 = 0.37. baseline 0.60 m는 실측(2026-09-05, 사용자 확인)이고,
+       -0.23은 위 base 안테나의 실측 x다. y=0, z=0.947은 base와 같다고 본 값이다 —
+       README의 배선 규약대로 두 안테나를 차량 세로축에 맞춰 같은 높이의 강체에
+       물렸다는 전제. 안테나를 서로 다른 높이에 달았다면 z를 따로 실측해서 고칠 것.
+       이 TF를 실제로 쓰는 곳: rover 드라이버가 /imu/heading(sensor_msgs/Imu)의
+       frame_id를 gps_rover_link로 찍고(rtk.launch.py), ekf_global의 imu1이 그걸
+       먹는다 — robot_localization이 IMU를 base_link_frame(body_link) 기준으로
+       돌려놓으려면 이 링크가 TF 트리에 있어야 한다. 없으면 base 안테나에서 났던
+       "Could not obtain body_link -> ... transform"과 같은 종류의 lookup 실패가 난다.
+       단 IMU에 실제로 적용되는 건 회전 성분뿐이고 여기 rpy는 0(= body_link와 같은
+       자세)이라, xyz를 틀리게 넣어도 헤딩 융합 결과는 바뀌지 않는다. xyz가 의미를
+       갖는 건 RViz 시각화와, 나중에 이 링크로 레버암 보정을 하게 될 때다.
+       sim에는 이 안테나가 없다 — gz navsat 센서는 gps_link 하나뿐이고(아래 "GPS
+       Sensor"), 시뮬레이션은 듀얼 안테나 헤딩을 흉내내지 않는다. 그래서 여기에는
+       대응하는 <gazebo> 센서 블록을 일부러 두지 않는다. -->
+  <joint name="gps_rover_joint" type="fixed">
+    <origin xyz="0.37 0 0.947" rpy="0 0 0"/>
+    <parent link="body_link"/>
+    <child link="gps_rover_link"/>
   </joint>
 <!-- LiDAR Fixed Joint -->

Commit message: TF Tree and Parameter Changes

File: src/control/hyper_control/urdf/vehicle.xacro (robot description, xacro)
@@ -61,4 +61,10 @@
   <xacro:property name="wheel_inertia_z" value="${1.0/2.0 * wheel_mass * wheel_radius * wheel_radius}"/>
   <xacro:property name="max_wheel_angular_velocity" value="${max_velocity / wheel_radius}"/>
+  <xacro:property name="antenna_height_from_ground" value="$(arg antenna_height_from_ground)"/>
+  <xacro:property name="car_body_origin_point_from_ground" value="$(arg car_body_origin_point_from_ground)"/>
+  <xacro:property name="lidar_height_from_ground" value="$(arg lidar_height_from_ground)"/>
+  <xacro:property name="rover_gps_offset_from_front_bumper" value="$(arg rover_gps_offset_from_front_bumper)"/>
+  <xacro:property name="gps_offset_from_front_bumper" value="$(arg gps_offset_from_front_bumper)"/>
+  <xacro:property name="lidar_offset_from_front_bumper" value="$(arg lidar_offset_from_front_bumper)" />
   <!-- Links -->
   <!-- Body Link -->
@@ -305,5 +311,5 @@
        내는 위치가 그만큼 통째로 움직입니다 — 실측 없이 건드리지 마세요. -->
   <joint name="gps_joint" type="fixed">
-    <origin xyz="-0.23 0 0.947" rpy="0 0 0"/>
+    <origin xyz="${body_length/2 + gps_offset_from_front_bumper} 0 ${antenna_height_from_ground - car_body_origin_point_from_ground}" rpy="0 0 0"/>
     <parent link="body_link"/>
     <child link="gps_link"/>
@@ -350,21 +356,10 @@
        대응하는 <gazebo> 센서 블록을 일부러 두지 않는다. -->
   <joint name="gps_rover_joint" type="fixed">
-    <origin xyz="0.37 0 0.947" rpy="0 0 0"/>
+    <origin xyz="${body_length/2 + rover_gps_offset_from_front_bumper} 0 ${antenna_height_from_ground - car_body_origin_point_from_ground}" rpy="0 0 0"/>
     <parent link="body_link"/>
     <child link="gps_rover_link"/>
   </joint>
-<!-- LiDAR Fixed Joint -->
-  <!-- 스캔 평면 높이 = wheel_radius*1.5 + body_height/2 + 이 오프셋
-       = 0.30 + 0.20 + 0.15 = 지면 위 0.65 m (parameters.yaml 기준값).
-       0.25 -> 0.15으로 10 cm 낮췄습니다. 이유:
-         - 이전 높이(0.75 m)는 hatchback 장애물 지붕(0.778 m)의 위쪽 2.8 cm를 스치기만 해서,
-           피치에 따라 반사가 들어왔다 말았다 했습니다(= local costmap이 비어 MPPI가 직진).
-           0.65 m면 지붕보다 12.8 cm 아래라 차체를 확실히 때립니다.
-         - 아래로는 차체 박스 윗면(0.50 m)보다 15 cm 위여야 gpu_lidar가 자기 차체에
-           가리지 않습니다.
-       주의: 이 xacro는 real.launch.py도 같이 씁니다. 실차 라이다를 실제로 0.65 m로
-       내려 달지 않으면 body_link->lidar_link TF가 실측과 어긋납니다. -->
   <joint name="lidar_joint" type="fixed">
-    <origin xyz="0.15 0 ${body_height/2 + 0.15}" rpy="0 0 0"/>
+    <origin xyz="${body_length/2 + lidar_offset_from_front_bumper} 0 ${lidar_height_from_ground - car_body_origin_point_from_ground}" rpy="0 0 0"/>
     <parent link="body_link"/>
     <child link="lidar_link"/>

Commit message: RPLIDAR A1 can only detect up to 1~2m range outdoors. Switching to RPP instead...

File: src/control/hyper_control/urdf/vehicle.xacro (robot description, xacro)
@@ -360,6 +360,11 @@
     <child link="gps_rover_link"/>
   </joint>
+  <!-- roll = PI: the unit is bolted to the bumper bracket upside down (top plate facing the
+       ground), so lidar_link's +Z points down and its +Y points to the vehicle's right. Without
+       this the scan is mirrored about the driving axis; an obstacle on the left is marked on
+       the right in the costmap. +X (the sensor's 0 deg mark) is the flip axis, so "forward" is
+       unchanged; if the bracket also turns the 0 deg mark, add the yaw here, not in the driver. -->
   <joint name="lidar_joint" type="fixed">
-    <origin xyz="${body_length/2 + lidar_offset_from_front_bumper} 0 ${lidar_height_from_ground - car_body_origin_point_from_ground}" rpy="0 0 0"/>
+    <origin xyz="${body_length/2 + lidar_offset_from_front_bumper} 0 ${lidar_height_from_ground - car_body_origin_point_from_ground}" rpy="${PI} 0 0"/>
     <parent link="body_link"/>
     <child link="lidar_link"/>
